File: EP-CC_CC_Eólica/EP-CC_CC_Eólica.kicad_sch (KiCad schematic)
At the start: 12 parts, among them J1 Screw_Terminal_01x03, J2 Screw_Terminal_01x02, Q1 Q_NIGBT_Diode_generic_GCE

Commit message: Skeleton
Parts:
- removed C1: C, symbol PCM_Elektuur:C
- added C2, C3: C-polar, Capacitor_THT:CP_Radial_D24.0mm_P10.00mm_SnapIn, symbol PCM_Elektuur:C-polar
- added C4: B32774D1155K000, Boost:CAP_B32774D1155K000_TDK, symbol Boost:B32774D1155K000
- added R1, R2: ROX3SJ100K, Boost:RES_ROX3S_TYCO_TYC, symbol Boost:ROX3SJ100K
- added STM1: ~, Boost:ST_Morpho_and_Zio_Connectors_144_STLink, symbol Custom:STM32
- added U1: LA100-P, Sensor_Current:LEM_LA25-P, symbol Sensor_Current:LA100-P
- added U2: LV25-P, Sensor_Voltage:LEM_LV25-P, symbol Sensor_Voltage:LV25-P
- CR1: renamed from D1; value D -> STBR3012W; footprint (none) -> Boost:DO-247_STM; symbol Device:D -> Boost:STBR3012W
- CR2: renamed from D2; value D -> STBR3012W; footprint (none) -> Boost:DO-247_STM; symbol Device:D -> Boost:STBR3012W
- CR3: renamed from D3; value D -> STBR3012W; footprint (none) -> Boost:DO-247_STM; symbol Device:D -> Boost:STBR3012W
- CR4: renamed from D4; value D -> STBR3012W; footprint (none) -> Boost:DO-247_STM; symbol Device:D -> Boost:STBR3012W
- CR5: renamed from D5; value D -> STBR3012W; footprint (none) -> Boost:DO-247_STM; symbol Device:D -> Boost:STBR3012W
- CR6: renamed from D6; value D -> STBR3012W; footprint (none) -> Boost:DO-247_STM; symbol Device:D -> Boost:STBR3012W
- D7: value D -> C4D20120D; footprint (none) -> Boost:TO-247-3_CRW; symbol Device:D -> Boost:C4D20120D
- J1: footprint (none) -> Connector_Phoenix_SPT:PhoenixContact_SPT_2.5_3-H-5.0-EX_1x03_P5.0mm_Horizontal
- J2: footprint (none) -> Connector_Phoenix_SPT:PhoenixContact_SPT_2.5_2-H-5.0-EX_1x02_P5.0mm_Horizontal
- L1: footprint (none) -> Inductor_THT:L_Axial_L26.0mm_D11.0mm_P7.62mm_Vertical_Fastron_77A
- Q1: value Q_NIGBT_Diode_generic_GCE -> IKW40N120H3; footprint (none) -> Boost:INF-PG-TO247-3; symbol PCM_Transistor_IGBT_AKL:Q_NIGBT_Diode_generic_GCE -> Boost:IKW40N120H3; Manufacturer (none) -> Infineon Technologies; Manufacturer Order Number (none) -> IKW40N120H3; PackageReference (none) -> PG-TO247-3-41
Connections:
- net Earth: now also CR1.2, CR3.2, CR5.2, C3.2 (-), C4.2, R2.2, U2.3 (HV-); no longer CR2.2 (A), CR4.2 (A), CR6.2 (A)
- net FAN_A: now also CR5.1, CR6.2; no longer CR1.2 (A), CR2.1 (K)
- net FAN_B: now also CR3.1, CR4.2; no longer CR3.2 (A), CR4.1 (K)
- net FAN_C: now also CR1.1, CR2.2; no longer CR5.2 (A), CR6.1 (K)
- net RECT+: now also CR2.1, CR4.1, CR6.1; no longer CR1.1 (K), CR3.1 (K), CR5.1 (K)
- net IGBT+: now reaches L1.2 (-), Q1.2 (COLLECTOR)
- net IGBT+: now also D7.1, D7.3; no longer D7.2 (A)
- net BOOST+: now reaches J2.1 (Pin_1)
- net BOOST+: now also D7.2, C2.1 (+), C4.1, R1.1, U2.1 (HV+); no longer D7.1 (K)
- new net 3V3: STM1.3V3 (+3V3), U1.3 (+), U2.5 (V+)
- new net CAP_MID: C2.2 (-), C3.1 (+)
- new net GND: STM1.GND, U1.2 (-), U2.6 (V-)
- new net R_MID: R1.2, R2.1
- new net STM_I: U1.1 (M)
- new net STM_V: U2.4 (M)
Other:
- moved on the sheet: J2

Commit message: 26/10/19
Parts:
- removed C3: C-polar, Capacitor_THT:CP_Radial_D24.0mm_P10.00mm_SnapIn, symbol PCM_Elektuur:C-polar
- removed CR1, CR2, CR3, CR4, CR5, CR6: STBR3012W, Boost:DO-247_STM, symbol Boost:STBR3012W
- removed D7: C4D20120D, Boost:TO-247-3_CRW, symbol Boost:C4D20120D
- removed R1, R2: ROX3SJ100K, Boost:RES_ROX3S_TYCO_TYC, symbol Boost:ROX3SJ100K
- removed U1: LA100-P, Sensor_Current:LEM_LA25-P, symbol Sensor_Current:LA100-P
- added C1: 470uF 200V, Boost:CAP_22 X 35_NCH, symbol Boost:LGU2D471MELZ
- added C2: 1.5uF 1.3KVDC, Boost:CAP_B32774D1155K000_TDK, symbol Boost:B32774D1155K000
- added Cdc1: 1uF, Capacitor_THT:CP_Radial_D5.0mm_P2.00mm, symbol PCM_Elektuur:C-polar
- added Cfilt1, Cref1, Cvcc1: 47nF - Cer, Capacitor_THT:C_Disc_D5.1mm_W3.2mm_P5.00mm, symbol PCM_SL_Devices:Capacitor_NP
- added Chcpl1, Chcpl2: 0.1uF - Cer, Capacitor_THT:C_Disc_D5.1mm_W3.2mm_P5.00mm, symbol PCM_SL_Devices:Capacitor_NP
- added Cprot1, Cprot2: 10n, Capacitor_THT:C_Disc_D6.0mm_W2.5mm_P5.00mm, symbol PCM_Elektuur:C
- added D1: 600V 35A, Boost:VS-36MT160, symbol Boost:VS-36MT160
- added D2, D3: C3D10060A, PCM_Package_TO_SOT_THT_AKL:TO-220-2_Vertical_KA, symbol PCM_Diode_Schottky_AKL:C3D10060A
- added DZ1: 15, Diode_THT:D_DO-27_P5.08mm_Vertical_AnodeUp, symbol PCM_Diode_Zener_AKL:D_Zener_Generic
- added DZprot1, DZprot2: 15, Diode_THT:D_DO-34_SOD68_P10.16mm_Horizontal, symbol PCM_Diode_Zener_AKL:D_Zener_Generic
- added Dhcpl1, Dhcpl2: 1.8V, LED_THT:LED_D5.0mm, symbol PCM_SL_Devices:LED
- added JSource1: Screw_Terminal_01x02, Boost:CONN2_2604-3102_WAG, symbol Connector:Screw_Terminal_01x02
- added L2: 311uH 15A, Boost:SHBC24W-2R1A0311V, symbol PCM_Elektuur:L
- added OCiso1, OCiso2: HCPL-3120, PCM_Package_DIP_AKL:DIP-8_W7.62mm_LongPads, symbol PCM_Optocoupler_Gate_Driver_AKL:HCPL-3120
- added Qbridge2: 600V40A, Boost:TO-220_High, symbol Boost:STGW60V60DF
- added Rg1, Rg2: 22, Resistor_THT:R_Axial_DIN0309_L9.0mm_D3.2mm_P2.54mm_Vertical, symbol PCM_SL_Resistors:Resistor
- added Rgs1, Rgs2, Rocd1: 10k, Resistor_THT:R_Axial_DIN0309_L9.0mm_D3.2mm_P2.54mm_Vertical, symbol PCM_SL_Resistors:Resistor
- added Rhcpl1, Rhcpl2: 180, Resistor_THT:R_Axial_DIN0309_L9.0mm_D3.2mm_P2.54mm_Vertical, symbol PCM_SL_Resistors:Resistor
- added Rled1, Rled2: 330, Resistor_THT:R_Axial_DIN0309_L9.0mm_D3.2mm_P2.54mm_Vertical, symbol PCM_SL_Resistors:Resistor
- added Rsafety1, Rsafety2: 4.7k, Boost:TWM20J4K7E, symbol PCM_Resistor_US_AKL:R_Power_L75.0mm_W9.0mm_P81.28mm
- added S1: HE/OL 25A, Boost:HO 25-N_SP33-1000, symbol Boost:HO_25-NP_SP33-1000
- added U2: LV25-P, Sensor_Voltage:LEM_LV25-P, symbol Sensor_Voltage:LV25-P
- added Upot1: MEV1S1515SC, Library:MEV1S1505SC, symbol Converter_DCDC:MEE1S1515SC
- C3: renamed from C2; value C-polar -> 470uF 200V; footprint Capacitor_THT:CP_Radial_D24.0mm_P10.00mm_SnapIn -> Boost:CAP_22 X 35_NCH; symbol PCM_Elektuur:C-polar -> Boost:LGU2D471MELZ
- C4: value B32774D1155K000 -> 1.5UF 1.3KVDC
- L1: value L -> 311uH 15A; footprint Inductor_THT:L_Axial_L26.0mm_D11.0mm_P7.62mm_Vertical_Fastron_77A -> Boost:SHBC24W-2R1A0311V
- Qbridge1: renamed from Q1; value IKW40N120H3 -> 600V40A; footprint Boost:INF-PG-TO247-3 -> Boost:TO-220_High; symbol Boost:IKW40N120H3 -> Boost:STGW60V60DF; Price (none) -> 1.3386
- renumbered U2 to U1
Connections:
- net CAP_MID is gone; now on net Earth: C3.2
- net STM_V is gone; now on net STM_Vin: U1.4 (M)
- net BOOST+: now also J2.2 (Pin_2), D2.1 (K), D3.1 (K), Rsafety2.1, U2.1 (HV+); no longer J2.1 (Pin_1), U1.1 (HV+)
- net Earth: now also J2.1 (Pin_1), C1.2, C2.2, Cdc1.2 (-), Chcpl1.2, Chcpl2.2, Cprot1.2 (-), Cprot2.2 (-), D1.5 (-), DZprot1.2 (A), DZprot2.2 (A), OCiso1.5 (GND), OCiso2.5 (GND), Qbridge2.3 (E), Rgs1.1, Rgs2.1, Rsafety1.2, Rsafety2.2, U2.3 (HV-), Upot1.5 (-Vout); no longer J2.2 (Pin_2)
- net FAN_A: now also D1.2 (AC)
- net FAN_B: now also D1.3 (AC)
- net FAN_C: now also D1.4 (AC)
- net GND: now also Cfilt1.2, Cref1.2, Cvcc1.1, DZ1.2 (A), JSource1.2 (Pin_2), Rocd1.1, S1.2 (GND), S1.7 (N/A), U2.6 (V-), Upot1.2 (-Vin)
- net RECT+: now also U1.1 (HV+), D1.1 (+), S1.11 (OUT); no longer L1.1 (+)
- net STM_Vref: now reaches STM1.PA4
- net STM_Vref: now also Cref1.1, S1.4 (Vref)
- net STM_Iin: now reaches STM1.PA5
- net STM_Iin: now also Cfilt1.1, S1.3 (Vout)
- net STM_Vin: now reaches STM1.PA6
- net STM_OCD: now reaches STM1.PB12
- net STM_OCD: now also Rocd1.2, S1.5 (OCD)
- net STM_S2: now reaches STM1.PE11
- net STM_S2: now also Dhcpl2.1, OCiso2.3
- net STM_S1: now reaches STM1.PE9
- net STM_S1: now also Dhcpl1.1, OCiso1.3
- net STM_Vout: now reaches STM1.PF9
- net STM_Vout: now also U2.4 (M)
- net 3V3 renamed +3.3V
- net +3.3V: now also Cvcc1.2, Rhcpl1.2, Rhcpl2.2, Rled1.2, Rled2.2, S1.1 (Vcc), U2.5 (V+)
- net IGBT+ renamed IGBT1+
- net IGBT1+: now also D2.2 (A), Qbridge2.2 (C); no longer Qbridge1.2 (COLLECTOR)
- net STM_IGBT renamed S1
- net S1: now also Cprot1.1 (+), DZprot1.1 (K), Rg1.1, Rgs1.2
- new net 15V: DZ1.1 (K), JSource1.1 (Pin_1), Upot1.1 (+Vin)
- new net IGBT2+: D3.2 (A), L2.2 (-), Qbridge1.2 (C)
- new net L+: C1.1, C2.1, L1.1 (+), L2.1 (+), Rsafety1.1, S1.8 (IN), S1.9 (IN)
- new net S2: Cprot2.1 (+), DZprot2.1 (K), Qbridge2.1 (G), Rg2.1, Rgs2.2
- new net V1: OCiso1.6, OCiso1.7, Rg1.2
- new net V2: OCiso2.6, OCiso2.7, Rg2.2
- new net Vcc_Pot: Cdc1.1 (+), Chcpl1.1, Chcpl2.1, OCiso1.8 (VCC), OCiso2.8 (VCC), Upot1.7 (+Vout)
- new net Vhcpl1: OCiso1.2, Rhcpl1.1
- new net Vhcpl2: OCiso2.2, Rhcpl2.1
- new net Vled1: Dhcpl1.2, Rled1.1
- new net Vled2: Dhcpl2.2, Rled2.1
- new net Winding: S1.10 (IN), S1.12 (OUT), S1.13 (OUT)
Other:
- moved on the sheet: C4, J1, J2, STM1, U1

Commit message: 26_10_21
Parts:
- added C5: 470UF 250V, Boost:LGW2E471MELZ40, symbol Boost:LGW2E471MELZ40
- added CFs1, CFs2, CFs3, CFs4: 1uF - Cer, Capacitor_THT:C_Disc_D7.5mm_W4.4mm_P5.00mm, symbol PCM_Elektuur:C
- added RFs1, RFs2, RFs3, RFs4: 1k, Resistor_THT:R_Axial_DIN0309_L9.0mm_D3.2mm_P2.54mm_Vertical, symbol PCM_Elektuur:R
- C1, C3: value 470uF 200V -> 470UF 250V; footprint Boost:CAP_22 X 35_NCH -> Boost:LGW2E471MELZ40; symbol Boost:LGU2D471MELZ -> Boost:LGW2E471MELZ40
Connections:
- net BOOST+: now also C5.1
- net Earth: now also C5.2
- net GND: now also CFs1.2 (-), CFs2.2 (-), CFs3.2 (-), CFs4.2 (-)
- net STM_Iin: now also RFs2.2 (-); no longer STM1.PA5
- net STM_Vin: now also RFs1.2 (-); no longer STM1.PA6
- net STM_Vout: now also RFs4.2 (-); no longer STM1.PF9
- net STM_Vref: now also RFs3.2 (-); no longer STM1.PA4
- new net Filt_Iin: CFs2.1 (+), RFs2.1 (+), STM1.PA5
- new net Filt_Vin: CFs1.1 (+), RFs1.1 (+), STM1.PA6
- new net Filt_Vout: CFs4.1 (+), RFs4.1 (+), STM1.PF9
- new net Filt_Vref: CFs3.1 (+), RFs3.1 (+), STM1.PA4
Other:
- moved on the sheet: C4, J2, Rsafety2, U2
